Commit message: Updated gps gazebo driver, fixed topic name issue

File: robotnik_sensors/urdf/gps.urdf.xacro (robot description, xacro)
@@ -1,18 +1,23 @@
 <?xml version="1.0"?>
 <robot name="sensor_gps" xmlns:xacro="http://wiki.ros.org/xacro">
-  <!-- if no latitude/longitud is specified, then use Fuente del Jarro as default -->
-  <xacro:macro name="sensor_gps" params="prefix parent *origin gps_latitude:=^|39.5080331 gps_longitude:=^|-0.4619816 update_rate:=^|5">
-	  <!-- ANTENNA GPS -->
-	  <joint name="${prefix}_joint" type="fixed">
-	    <axis xyz="0 1 0"/>
+	<xacro:macro name="sensor_gps"
+               params="prefix
+                       parent
+                       *origin
+                       simulation:=false
+                       node_name:=gps
+                       node_namespace:=${None}
+                       topic_prefix:=~/
+                       update_rate:=5.0">
+	  <joint name="${prefix}joint" type="fixed">
 	    <xacro:insert_block name="origin"/>
 	    <parent link="${parent}"/>
-	    <child link="${prefix}_base_link"/>
+	    <child link="${prefix}base_link"/>
 	  </joint>
-	  <link name="${prefix}_base_link">
-		<inertial>
-			<origin xyz="0.0 0 0.015" rpy="0 0 0" />
-			<mass value="0.2" />
-			<xacro:solid_cuboid_inertia m="0.2" w="0.081" h="0.081" d="0.03" />
+	  <link name="${prefix}base_link">
+      <inertial>
+        <origin xyz="0.0 0 0.015" rpy="0 0 0" />
+        <mass value="0.2" />
+        <xacro:solid_cuboid_inertia m="0.2" w="0.081" h="0.081" d="0.03" />
       </inertial>
 	    <visual>
@@ -22,5 +27,5 @@
         </material>
 	      <geometry>
-	        <mesh filename="package://robotnik_sensors/meshes/antenna_3GO16.stl" scale="1.0 1.0 1.0"/>
+	        <mesh filename="package://robotnik_sensors/meshes/antenna_3GO16.stl"/>
 	      </geometry>
 	    </visual>
@@ -28,35 +33,55 @@
 	      <origin rpy="0 0 0" xyz="0 0 0"/>
 	      <geometry>
-	        <mesh filename="package://robotnik_sensors/meshes/antenna_3GO16.stl" scale="1.0 1.0 1.0"/>
+	        <mesh filename="package://robotnik_sensors/meshes/antenna_3GO16.stl"/>
 	      </geometry>
 	    </collision>
 	  </link>
-	  <gazebo reference="${prefix}_base_link">
+	  <gazebo reference="${prefix}base_link">
 	    <material>Gazebo/White</material>
 	    <gravity>true</gravity>
 	  </gazebo>
-    <gazebo>
-      <plugin name="${prefix}_controller" filename="libhector_gazebo_ros_gps.so">
-        <alwaysOn>1</alwaysOn>
-        <updateRate>${update_rate}</updateRate>
-        <bodyName>${prefix}_base_link</bodyName> <!-- must be the link of the gps device, not the base_link or base_footprint -->
-        <frameId>${prefix}_base_link</frameId>
-        <topicName>gps/fix</topicName>
-        <!-- GPS coordinates -->
-        <referenceLatitude>${gps_latitude}</referenceLatitude>
-        <referenceLongitude>${gps_longitude}</referenceLongitude>
-        <!-- To set heading in ENU orientation (degrees) -->
-        <referenceHeading>90</referenceHeading>
-        <velocityTopicName>gps/fix_velocity</velocityTopicName>
-        <drift>0.0 0.0 0.0</drift>
-        <!--<drift>0.0001 0.0001 0.0001</drift>-->
-        <!--<drift>0.3 0.3 0.3</drift>-->
-        <gaussianNoise>0.00001 0.00001 0.00001</gaussianNoise>
-        <!--<gaussianNoise>0.00001 0.00001 0.00001</gaussianNoise>-->
-        <velocityDrift>0.00001 0.00001 0.00001</velocityDrift>
-        <!--<velocityGaussianNoise>0.1 0.1 0.1</velocityGaussianNoise>-->
-        <velocityGaussianNoise>0.00001 0.00001 0.00001</velocityGaussianNoise>
-      </plugin>
-	</gazebo>
+    <gazebo reference="${prefix}base_link">
+      <sensor type="gps" name="${prefix}sensor">
+        <always_on>true</always_on>
+        <update_rate>${update_rate}</update_rate>
+        <gps>
+          <position_sensing>
+            <horizontal>
+              <noise type="gaussian">
+                <mean>0.0</mean>
+                <stddev>0.1</stddev>
+              </noise>
+            </horizontal>
+            <vertical>
+              <noise type="gaussian">
+                <mean>0.0</mean>
+                <stddev>0.1</stddev>
+              </noise>
+            </vertical>
+          </position_sensing>
+          <vertical_sensing>
+            <horizontal>
+              <noise type="gaussian">
+                <mean>0.0</mean>
+                <stddev>0.1</stddev>
+              </noise>
+            </horizontal>
+            <vertical>
+              <noise type="gaussian">
+                <mean>0.0</mean>
+                <stddev>0.1</stddev>
+              </noise>
+            </vertical>
+          </vertical_sensing>
+        </gps>
+        <plugin name="${node_name}" filename="libgazebo_ros_gps_sensor.so">
+          <ros>
+            <namespace>${node_namespace}</namespace>
+            <remapping>~/out:=${topic_prefix}/fix</remapping>
+            <remapping>~/vel:=${topic_prefix}/vel</remapping>
+          </ros>
+        </plugin>
+      </sensor>
+	  </gazebo>
   </xacro:macro>
 </robot>
