Commit message: added node_name param, fixed topic name parameter of the gazebo driver

File: robotnik_sensors/urdf/rs_bpearl.urdf.xacro (robot description, xacro)
@@ -2,5 +2,5 @@
 <robot name="sensor_rs_bpearl" xmlns:xacro="http://wiki.ros.org/xacro">
   <xacro:property name="M_PI" value="3.1415926535897931" />
-  <xacro:macro name="sensor_rs_bpearl" params="prefix parent prefix_topic *origin range_min range_max hfov samples vfov lasers fps gpu:=true">
+  <xacro:macro name="sensor_rs_bpearl" params="prefix parent prefix_topic node_name *origin range_min range_max hfov samples vfov lasers fps gpu:=true">
     <joint name="${prefix}_base_joint" type="fixed">
       <xacro:insert_block name="origin" />
@@ -38,7 +38,7 @@
     </joint>
     <link name="${prefix}_link"/>
-    <xacro:sensor_rs_bpearl_gazebo prefix="${prefix}" range_min="${range_min}" range_max="${range_max}" hfov="${hfov}" samples="${samples}" vfov="${vfov}" lasers="${lasers}" fps="${fps}" gpu="${gpu}"/>
+    <xacro:sensor_rs_bpearl_gazebo prefix="${prefix}" prefix_topic="${prefix_topic}" node_name="${node_name}" range_min="${range_min}" range_max="${range_max}" hfov="${hfov}" samples="${samples}" vfov="${vfov}" lasers="${lasers}" fps="${fps}" gpu="${gpu}"/>
   </xacro:macro>
-  <xacro:macro name="sensor_rs_bpearl_gazebo" params="prefix range_min range_max hfov samples vfov lasers fps gpu">
+  <xacro:macro name="sensor_rs_bpearl_gazebo" params="prefix prefix_topic node_name range_min range_max hfov samples vfov lasers fps gpu">
     <gazebo reference="${prefix}_base_link">
       <visual>
@@ -96,5 +96,8 @@
           </ray>
           <plugin name="${prefix}_controller" filename="${plugin_lib}">
-            <topicName>${prefix_topic}/points</topicName>
+          <ros>
+            <namespace>${node_name}</namespace>
+            <remapping>~/out:=${prefix_topic}/points</remapping>
+          </ros>
             <gaussian_noise>0.008</gaussian_noise>
             <organize_cloud>0</organize_cloud>
