Commit message: improving sensor colors

File: robotnik_sensors/urdf/3d_lidar/robosense_helios_16p.urdf.xacro (robot description, xacro)
@@ -40,4 +40,8 @@
       </inertial>
     </link>
+    <gazebo reference="${frame_prefix}base_link">
+        <material>Gazebo/Grey</material>
+        <gravity>true</gravity>
+    </gazebo>
     <joint name="${frame_prefix}joint" type="fixed">
       <parent link="${frame_prefix}base_link"/>

File: robotnik_sensors/urdf/gps/ublox.urdf.xacro (robot description, xacro)
@@ -47,7 +47,7 @@
 	  </link>
 	<gazebo reference="${frame_prefix}base_link">
-	    <material>Gazebo/White</material>
+	    <material>Gazebo/Grey</material>
 	    <gravity>true</gravity>
-	  </gazebo>
+	</gazebo>
     <xacro:if value="${simulation}">
 		<gazebo reference="${frame_prefix}base_link">

Commit message: filtered point cloud for robosense

File: robotnik_sensors/urdf/3d_lidar/robosense_helios_16p.urdf.xacro (robot description, xacro)
@@ -37,10 +37,10 @@
         <mass value="0.840" />
         <origin xyz="0 0 0.04135" />
-		<xacro:solid_cuboid_inertia m="0.840" w="0.109" h="0.109" d="0.0827" />
+        <xacro:solid_cuboid_inertia m="0.840" w="0.109" h="0.109" d="0.0827" />
       </inertial>
     </link>
     <gazebo reference="${frame_prefix}base_link">
-        <material>Gazebo/Grey</material>
-        <gravity>true</gravity>
+      <material>Gazebo/Grey</material>
+      <gravity>true</gravity>
     </gazebo>
     <joint name="${frame_prefix}joint" type="fixed">
@@ -55,54 +55,61 @@
   </xacro:macro>
   <xacro:macro name="sensor_robosense_helios_16p_gazebo">
-      <xacro:if value="${gpu}">
-        <xacro:property name="ray_type" value="gpu_ray" />
-      </xacro:if>
-      <xacro:unless value="${gpu}">
-        <xacro:property name="ray_type" value="ray" />
-      </xacro:unless>
-      <gazebo reference="${frame_prefix}link">
-        <sensor type="${ray_type}" name="${frame_prefix}sensor">
-          <pose>0 0 0 0 0 0</pose>
-          <visualize>false</visualize>
-          <update_rate>10</update_rate>
-          <ray>
-            <scan>
-              <horizontal>
-                <samples>1200</samples>
-                <resolution>1.0</resolution>
-                <min_angle>${-radians(180)}</min_angle>
-                <max_angle>${radians(180)}</max_angle>
-              </horizontal>
-              <vertical>
-                <samples>32</samples>
-                <resolution>1.0</resolution>
-                <min_angle>0.0</min_angle>
-                <max_angle>${radians(85)}</max_angle>
-              </vertical>
-            </scan>
-            <range>
-              <min>0.10</min>
-              <max>50</max>
-              <resolution>0.001</resolution>
-            </range>
-            <noise>
-              <type>gaussian</type>
-              <mean>0.0</mean>
-              <stddev>0.00</stddev>
-            </noise>
-          </ray>
-          <plugin name="${node_name}" filename="libgazebo_ros_velodyne_laser.so">
-            <ros>
-              <namespace>${node_namespace}</namespace>
-              <remapping>~/out:=${topic_prefix}point_cloud</remapping>
-            </ros>
-            <frame_name>${frame_prefix}link</frame_name>
-            <min_range>0.5</min_range>
-            <max_range>100.0</max_range>
-            <gaussian_noise>0.01</gaussian_noise>
-            <organize_cloud>0</organize_cloud>
-          </plugin>
-        </sensor>
-      </gazebo>
+    <xacro:if value="${gpu}">
+      <xacro:property name="ray_type" value="gpu_ray" />
+    </xacro:if>
+    <xacro:unless value="${gpu}">
+      <xacro:property name="ray_type" value="ray" />
+    </xacro:unless>
+    <gazebo reference="${frame_prefix}link">
+      <sensor type="${ray_type}" name="${frame_prefix}sensor">
+        <pose>0 0 0 0 0 0</pose>
+        <visualize>false</visualize>
+        <update_rate>10</update_rate>
+        <ray>
+          <scan>
+            <horizontal>
+              <samples>1200</samples>
+              <resolution>1.0</resolution>
+              <min_angle>${-radians(180)}</min_angle>
+              <max_angle>${radians(180)}</max_angle>
+            </horizontal>
+            <vertical>
+              <samples>32</samples>
+              <resolution>1.0</resolution>
+              <min_angle>0.0</min_angle>
+              <max_angle>${radians(85)}</max_angle>
+            </vertical>
+          </scan>
+          <range>
+            <min>0.10</min>
+            <max>50</max>
+            <resolution>0.001</resolution>
+          </range>
+          <noise>
+            <type>gaussian</type>
+            <mean>0.0</mean>
+            <stddev>0.00</stddev>
+          </noise>
+        </ray>
+        <plugin name="${node_name}" filename="libgazebo_ros_velodyne_laser.so">
+          <ros>
+            <namespace>${node_namespace}</namespace>
+            <remapping>~/out:=${topic_prefix}points_filtered</remapping>
+            <qos>
+              <topic name="/robot/top_3d_laser/points_filtered">
+                <publisher>
+                  <reliability>best_effort</reliability>
+                </publisher>
+              </topic>
+            </qos>
+          </ros>
+          <frame_name>${frame_prefix}link</frame_name>
+          <min_range>0.5</min_range>
+          <max_range>100.0</max_range>
+          <gaussian_noise>0.01</gaussian_noise>
+          <organize_cloud>0</organize_cloud>
+        </plugin>
+      </sensor>
+    </gazebo>
   </xacro:macro>
 </robot>

Commit message: setting best effort qos for zed cameras and fixing robosense topic

File: robotnik_sensors/urdf/3d_lidar/robosense_helios_16p.urdf.xacro (robot description, xacro)
@@ -95,15 +95,8 @@
           <ros>
             <namespace>${node_namespace}</namespace>
-            <remapping>~/out:=${topic_prefix}points_filtered</remapping>
-            <qos>
-              <topic name="/robot/top_3d_laser/points_filtered">
-                <publisher>
-                  <reliability>best_effort</reliability>
-                </publisher>
-              </topic>
-            </qos>
+            <remapping>~/out:=${topic_prefix}points</remapping>
           </ros>
           <frame_name>${frame_prefix}link</frame_name>
-          <min_range>0.5</min_range>
+          <min_range>0.05</min_range>
           <max_range>100.0</max_range>
           <gaussian_noise>0.01</gaussian_noise>

File: robotnik_sensors/urdf/depth/stereolabs_generic.urdf.xacro (robot description, xacro)
@@ -22,11 +22,11 @@
     </xacro:if>
     <xacro:if value="${model == 'zed'}">
-        <xacro:property name="baseline" value="0.12" />
+      <xacro:property name="baseline" value="0.12" />
     </xacro:if>
     <xacro:if value="${model == 'zedm'}">
-        <xacro:property name="baseline" value="0.06" />
+      <xacro:property name="baseline" value="0.06" />
     </xacro:if>
     <xacro:if value="${model == 'zed2'}">
-        <xacro:property name="baseline" value="0.12" />
+      <xacro:property name="baseline" value="0.12" />
     </xacro:if>
     <joint name="${frame_prefix}base_joint" type="fixed">
@@ -36,5 +36,5 @@
     </joint>
     <link name="${frame_prefix}base_link">
-       <visual>
+      <visual>
         <origin xyz="0 0 0" rpy="0 0 0"/>
         <geometry>
@@ -57,5 +57,5 @@
       </inertial>
     </link>
-   <!-- Left camera -->
+    <!-- Left camera -->
     <joint name="${frame_prefix}color_left_joint" type="fixed">
       <origin xyz="0.0 0.06 0.0" rpy="0.0 0.0 0.0" />
@@ -196,4 +196,31 @@
               <remapping>~/depth/camera_info:=${topic_prefix}depth/camera_info</remapping>
               <remapping>~/depth/image_raw:=${topic_prefix}depth/depth_registered</remapping>
+              <qos>
+                <topic name="${topic_prefix}rgb/image_raw_color">
+                  <publisher>
+                    <reliability>best_effort</reliability>
+                  </publisher>
+                </topic>
+                <topic name="${topic_prefix}rgb/camera_info">
+                  <publisher>
+                    <reliability>best_effort</reliability>
+                  </publisher>
+                </topic>
+                <topic name="${topic_prefix}point_cloud/cloud_registered">
+                  <publisher>
+                    <reliability>best_effort</reliability>
+                  </publisher>
+                </topic>
+                <topic name="${topic_prefix}depth/camera_info">
+                  <publisher>
+                    <reliability>best_effort</reliability>
+                  </publisher>
+                </topic>
+                <topic name="${topic_prefix}depth/depth_registered">
+                  <publisher>
+                    <reliability>best_effort</reliability>
+                  </publisher>
+                </topic>
+              </qos>
             </ros>
             <camera_name>${node_name}</camera_name>
