Commit message: reducing gps noise

File: robotnik_sensors/urdf/gps/ublox.urdf.xacro (robot description, xacro)
@@ -10,89 +10,89 @@
 						topic_prefix:=~/
 						update_rate:=5.0">
-	  <!-- ANTENNA GPS -->
-	  <joint name="${frame_prefix}base_joint" type="fixed">
-	    <xacro:insert_block name="origin"/>
-	    <parent link="${parent}"/>
-	    <child link="${frame_prefix}base_link"/>
-	  </joint>
-	  <link name="${frame_prefix}base_link">
-		<inertial>
-			<origin xyz="0.0 0 0.015" rpy="0 0 0" />
-			<mass value="0.2" />
-			<xacro:solid_cuboid_inertia m="0.2" w="0.081" h="0.081" d="0.03" />
-      </inertial>
-	    <visual>
-	      <origin rpy="0 0 0" xyz="0 0 0"/>
-		  <material name="ublox_gps_color">
-           <color rgba="0.5 0.5 0.5 1"/>
-          </material>
-	      <geometry>
-	        <mesh filename="package://robotnik_sensors/meshes/gps/antenna_ANN_MB.stl" scale="1.0 1.0 1.0"/>
-	      </geometry>
-	    </visual>
-	    <collision>
-	      <origin rpy="0 0 0" xyz="0 0 0.01125"/>
-	        <geometry>
-	          <box size="0.0607 0.083 0.0225"/>
-	        </geometry>
-	    </collision>
+		<!-- ANTENNA GPS -->
+		<joint name="${frame_prefix}base_joint" type="fixed">
+			<xacro:insert_block name="origin"/>
+			<parent link="${parent}"/>
+			<child link="${frame_prefix}base_link"/>
+		</joint>
+		<link name="${frame_prefix}base_link">
+			<inertial>
+				<origin xyz="0.0 0 0.015" rpy="0 0 0" />
+				<mass value="0.2" />
+				<xacro:solid_cuboid_inertia m="0.2" w="0.081" h="0.081" d="0.03" />
+			</inertial>
+			<visual>
+				<origin rpy="0 0 0" xyz="0 0 0"/>
+				<material name="ublox_gps_color">
+					<color rgba="0.5 0.5 0.5 1"/>
+				</material>
+				<geometry>
+					<mesh filename="package://robotnik_sensors/meshes/gps/antenna_ANN_MB.stl" scale="1.0 1.0 1.0"/>
+				</geometry>
+			</visual>
+			<collision>
+				<origin rpy="0 0 0" xyz="0 0 0.01125"/>
+				<geometry>
+					<box size="0.0607 0.083 0.0225"/>
+				</geometry>
+			</collision>
+		</link>
+		<joint name="${frame_prefix}joint" type="fixed">
+			<axis xyz="1 0 0"/>
+			<origin xyz="0.0 0.0 0.01125"/>
+			<parent link="${frame_prefix}base_link"/>
+			<child link="${frame_prefix}link"/>
+		</joint>
+		<link name="${frame_prefix}link">
 	  </link>
-	  <joint name="${frame_prefix}joint" type="fixed">
-	      <axis xyz="1 0 0"/>
-	      <origin xyz="0.0 0.0 0.01125"/>
-	      <parent link="${frame_prefix}base_link"/>
-	      <child link="${frame_prefix}link"/>
-	  </joint>
-	  <link name="${frame_prefix}link">
-	  </link>
-	<gazebo reference="${frame_prefix}base_link">
-	    <material>Gazebo/Grey</material>
-	    <gravity>true</gravity>
-	</gazebo>
-    <xacro:if value="${simulation}">
 		<gazebo reference="${frame_prefix}base_link">
-		<sensor type="gps" name="${frame_prefix}sensor">
-			<always_on>true</always_on>
-			<update_rate>${update_rate}</update_rate>
-			<gps>
-			<position_sensing>
-				<horizontal>
-				<noise type="gaussian">
-					<mean>0.0</mean>
-					<stddev>0.1</stddev>
-				</noise>
-				</horizontal>
-				<vertical>
-				<noise type="gaussian">
-					<mean>0.0</mean>
-					<stddev>0.1</stddev>
-				</noise>
-				</vertical>
-			</position_sensing>
-			<vertical_sensing>
-				<horizontal>
-				<noise type="gaussian">
-					<mean>0.0</mean>
-					<stddev>0.1</stddev>
-				</noise>
-				</horizontal>
-				<vertical>
-				<noise type="gaussian">
-					<mean>0.0</mean>
-					<stddev>0.1</stddev>
-				</noise>
-				</vertical>
-			</vertical_sensing>
-			</gps>
-			<plugin name="${node_name}" filename="libgazebo_ros_gps_sensor.so">
-			<ros>
-				<namespace>${node_namespace}</namespace>
-				<remapping>~/out:=${topic_prefix}fix</remapping>
-				<remapping>~/vel:=${topic_prefix}vel</remapping>
-			</ros>
-			</plugin>
-		</sensor>
+			<material>Gazebo/Grey</material>
+			<gravity>true</gravity>
 		</gazebo>
-    </xacro:if>
-  </xacro:macro>
+		<xacro:if value="${simulation}">
+			<gazebo reference="${frame_prefix}base_link">
+				<sensor type="gps" name="${frame_prefix}sensor">
+					<always_on>true</always_on>
+					<update_rate>${update_rate}</update_rate>
+					<gps>
+						<position_sensing>
+							<horizontal>
+								<noise type="gaussian">
+									<mean>0.0</mean>
+									<stddev>0.0000001</stddev>
+								</noise>
+							</horizontal>
+							<vertical>
+								<noise type="gaussian">
+									<mean>0.0</mean>
+									<stddev>0.0000001</stddev>
+								</noise>
+							</vertical>
+						</position_sensing>
+						<vertical_sensing>
+							<horizontal>
+								<noise type="gaussian">
+									<mean>0.0</mean>
+									<stddev>0.0000001</stddev>
+								</noise>
+							</horizontal>
+							<vertical>
+								<noise type="gaussian">
+									<mean>0.0</mean>
+									<stddev>0.0000001</stddev>
+								</noise>
+							</vertical>
+						</vertical_sensing>
+					</gps>
+					<plugin name="${node_name}" filename="libgazebo_ros_gps_sensor.so">
+						<ros>
+							<namespace>${node_namespace}</namespace>
+							<remapping>~/out:=${topic_prefix}fix</remapping>
+							<remapping>~/vel:=${topic_prefix}vel</remapping>
+						</ros>
+					</plugin>
+				</sensor>
+			</gazebo>
+		</xacro:if>
+	</xacro:macro>
 </robot>
