Commit message: fixing myahrs imu

File: robotnik_sensors/urdf/imu/myahrs.urdf.xacro (robot description, xacro)
@@ -37,8 +37,8 @@
     </link>
     <joint name="${frame_prefix}joint" type="fixed">
-        <axis xyz="1 0 0"/>
-        <origin xyz="-0.00745 0.0 0.0088"/>
-        <parent link="${frame_prefix}base_link"/>
-        <child link="${frame_prefix}link"/>
+      <axis xyz="1 0 0"/>
+      <origin xyz="-0.00745 0.0 0.0088"/>
+      <parent link="${frame_prefix}base_link"/>
+      <child link="${frame_prefix}link"/>
     </joint>
     <link name="${frame_prefix}link" />
@@ -51,5 +51,5 @@
         <sensor name="${frame_prefix}sensor" type="imu">
           <always_on>true</always_on>
-          <update_rate>200</update_rate>
+          <update_rate>100</update_rate>
           <visualize>true</visualize>
           <imu>
@@ -118,5 +118,5 @@
             <ros>
               <namespace>${node_namespace}</namespace>
-              <remapping>~/out:=${topic_prefix}data</remapping>
+              <remapping>~/out:=${topic_prefix}data_raw</remapping>
             </ros>
             <initial_orientation_as_reference>false</initial_orientation_as_reference>
